File: StepperDriver.kicad_pcb (KiCad board)
At the start: 2 copper layers, 100 x 100 mm, 17 parts, among them J1 USB4105-GF-A, J2 10118193-0001LF, J2 USB_B_Micro, M1 Stepper_Motor_bipolar, U1 STSPIN220

Commit message: Updated Logo library reference
Parts:
- removed G***: LOGO, StepperDriver-footprints:AC_Logo
- added AC_LOGO: LOGO, AC-kicad-library:AC_Logo_17mm_20mm, F.Cu at (72.5, 134.8)

Commit message: update schematic image
Parts:
- removed the J2 at (91.0, 80.5)
- added J3: Conn_01x04_Socket, Connector_Molex:Molex_SL_171971-0004_1x04_P2.54mm_Vertical, F.Cu at (125.4, 93.5)
- added REF**: Molex_PicoBlade_53261-0471_1x04-1MP_P1.25mm_Horizontal, Connector_Molex:Molex_PicoBlade_53261-0471_1x04-1MP_P1.25mm_Horizontal, F.Cu at (109.8, 142.3)
- added REF**: TerminalBlock_Phoenix_MPT-0,5-4-2.54_1x04_P2.54mm_Horizontal, TerminalBlock_Phoenix:TerminalBlock_Phoenix_MPT-0,5-4-2.54_1x04_P2.54mm_Horizontal, F.Cu at (105.9, 133.2)
- added REF**: Hirose_FH12-6S-0.5SH_1x06-1MP_P0.50mm_Horizontal, Connector_FFC-FPC:Hirose_FH12-6S-0.5SH_1x06-1MP_P0.50mm_Horizontal, B.Cu at (109.8, 142.3)
- added SW3: RotaryEncoder_Switch_MP, Rotary_Encoder:RotaryEncoder_Alps_EC11E-Switch_Vertical_H20mm_CircularMountingHoles, F.Cu at (129.6, 74.0)
- moved M1 16.6 mm to (104.9, 69.2)
