File: StepperDriver.kicad_sch (KiCad schematic)
At the start: 15 parts, among them J1 USB4105-GF-A, J2 10118193-0001LF, M1 Stepper_Motor_bipolar, SW1 SW_Push, SW2 SW_Push, U1 STSPIN220

Commit message: update schematic image
Parts:
- added C1: C_Small, Capacitor_SMD:C_0603_1608Metric, symbol Device:C_Small
- added C2, Cen: 22nf, Capacitor_SMD:C_0603_1608Metric, symbol Device:C_Small
- added C3: 100nF, Capacitor_SMD:C_0603_1608Metric, symbol Device:C_Small
- added C4: 1uF, Capacitor_SMD:C_0603_1608Metric, symbol Device:C_Small
- added C5: 10uF, Capacitor_SMD:C_0603_1608Metric, symbol Device:C_Small
- added C6: 22uF, Capacitor_SMD:CP_Elec_4x3, symbol Device:C_Polarized_Small_US
- added J3: Conn_01x04_Socket, Connector_Molex:Molex_SL_171971-0004_1x04_P2.54mm_Vertical, symbol Connector:Conn_01x04_Socket
- added R3: 1K, Resistor_SMD:R_0603_1608Metric, symbol Device:R_Small
- added R5, R6: 330mR, Resistor_SMD:R_0603_1608Metric, symbol Device:R_Small
- added R8, Ren: 20K, Resistor_SMD:R_0603_1608Metric, symbol Device:R_Small
- added ROFF: 10K, Resistor_SMD:R_0603_1608Metric, symbol Device:R_Small
- added SW4: RotaryEncoder_Switch_MP, Rotary_Encoder:RotaryEncoder_Alps_EC12E-Switch_Vertical_H20mm_CircularMountingHoles, symbol Device:RotaryEncoder_Switch_MP
- D1, D2, D3: footprint LED_SMD:LED_0603_1608Metric_Pad1.05x0.95mm_HandSolder -> StepperDriver-footprints:LED_0603_1608Metric_Pad1.05x0.95mm_HandSolder
- H1, H2, H3, H4: footprint MountingHole:MountingHole_3.2mm_M3_Pad_Via -> StepperDriver-footprints:MountingHole_3.2mm_M3_Pad_Via
- J1: footprint Connector_USB:USB_C_Receptacle_GCT_USB4105-xx-A_16P_TopMnt_Horizontal -> StepperDriver-footprints:USB_C_Receptacle_GCT_USB4105-xx-A_16P_TopMnt_Horizontal
- J2: footprint AC-kicad-library:MICRO-USB-SMD_10118193-0001LF -> StepperDriver-footprints:MICRO-USB-SMD_10118193-0001LF
- M1: footprint TerminalBlock:TerminalBlock_Xinya_XY308-2.54-4P_1x04_P2.54mm_Horizontal -> StepperDriver-footprints:TerminalBlock_Xinya_XY308-2.54-4P_1x04_P2.54mm_Horizontal
- R1, R2: footprint Resistor_SMD:R_0603_1608Metric_Pad0.98x0.95mm_HandSolder -> StepperDriver-footprints:R_0603_1608Metric_Pad0.98x0.95mm_HandSolder
- U1: footprint Package_DFN_QFN:VQFN-16-1EP_3x3mm_P0.5mm_EP1.68x1.68mm -> StepperDriver-footprints:VQFN-16-1EP_3x3mm_P0.5mm_EP1.68x1.68mm
Connections:
- net DIR: now reaches U1.1 (DIR)
- net B1: now reaches U1.10 (OUTB1)
- net VREF: now reaches U1.11 (REF)
- net TOFF: now reaches U1.12 (TOFF)
- net TOFF: now also R3.1, ROFF.1
- net FAULT_MCU: now reaches U1.13 (EN/FLT)
- net FAULT_MCU: now also Cen.1, Ren.2
- net at U1.14 (STBY/RESET): now also R8.2
- net MODE2: now reaches U1.15 (MODE2)
- net MODE1: now reaches U1.16 (MODE1)
- net Earth: now reaches U1.17 (EPAD)
- net Earth: now also U1.7 (GND), C2.2, C3.2, C4.2, C5.2, C6.2, Cen.2, R5.2, R6.1, ROFF.2
- net STEP: now reaches U1.2 (STCK)
- net A1: now reaches U1.3 (OUTA1)
- net at U1.4 (SENSEA): now also R6.2
- net A2: now reaches U1.5 (OUTA2)
- net VMOT: now reaches U1.6 (VS)
- net VMOT: now also C3.1, C4.1, C5.1, C6.1
- net B2: now reaches U1.8 (OUTB2)
- net at U1.9 (SENSEB): now also R5.1
- new net: C2.1, R3.2
- new net EN_MCU: Ren.1
- new net STBY: R8.1
Other:
- note added: "Check If seperate VCC and VMOT needed"
- note added: "Check Required Capacitance and if electrolytics needed"
- note added: "VMOT: 1.8V -10V IMot: 1.3A"
- note added: "VRef Recommended: 0.1V-0.5V"
